File: projects/attiny13a-buffered-electrical-bypass-quasi-ic/attiny13a-quasi-ic.kicad_pcb (KiCad board)
At the start: 2 copper layers, 35 x 23 mm, 45 parts, among them J3 Conn_02x06_Buf_Byp_Module, Q3 2N7002, U1 OPA1678IDRGR, U4 AP7375-50SA-7, U6 ATTINY13A-SSUR, U9 TMUX4053DYYR

Commit message: add copyright and license
Other:
- board text added: "© 2026 Matthew Garman CERN-OHL-P-2.0 https://github.com/matt-garman/mcu-bypass-hardware"
Changed lines of the file:
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@@
+		)
+	)
+	(gr_text "© 2026 Matthew Garman\nCERN-OHL-P-2.0\nhttps://github.com/matt-garman/mcu-bypass-hardware"
+		(at 193.75 133.25 0)
+		(layer "B.SilkS")
+		(effects
+			(font
+				(size 1 0.75)
+				(thickness 0.14)
+				(bold yes)
+			)
+			(justify left bottom mirror)
 		)
 	)
