File: projects/attiny13a-buffered-electrical-bypass-quasi-ic/attiny13a-quasi-ic.kicad_sch (KiCad schematic)
At the start: 45 parts, among them J3 Conn_02x06_Buf_Byp_Module, Q3 2N7002, U1 OPA1678IDRGR, U4 AP7375-50SA-7, U6 ATTINY13A-SSUR, U9 TMUX4053DYYR

Commit message: add copyright and license
Other:
- title: (none) -> ATtiny13a Buffered Electrical Bypass Quasi-IC
Changed lines of the file:
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@@
 	(generator_version "10.0")
 	(paper "A4")
+	(title_block
+		(title "ATtiny13a Buffered Electrical Bypass Quasi-IC")
+		(rev "1.0")
+		(comment 1 "SPDX-License-Identifier: CERN-OHL-P-2.0")
+		(comment 2 "© 2026 Matthew Garman")
+		(comment 3 "https://github.com/matt-garman/mcu-bypass-hardware")
+	)
 	(text "PARENT PCB INTERFACE"
 		(exclude_from_sim no)
